Commit message: Error en los sensores

File: create3_sim/irobot_create_common/irobot_create_description/urdf/create3.urdf.xacro (robot description, xacro)
@@ -267,3 +267,56 @@
     </gazebo>
   </xacro:if>
+  <!-- LIDAR -->
+  <!-- NO FUNCIONA
+  <link name="laser_frame">
+      <visual>
+          <geometry>
+              <cylinder radius="0.05" length="0.04"/>
+          </geometry>
+          <material name="red"/>
+      </visual>
+      <collision>
+          <geometry>
+              <cylinder radius="0.05" length="0.04"/>
+          </geometry>
+      </collision>
+      <xacro:inertial_cylinder mass="0.1" length="0.04" radius="0.05">
+          <origin xyz="0 0 0" rpy="0 0 0"/>
+      </xacro:inertial_cylinder>
+  </link>
+  <joint name="laser_joint" type="fixed">
+    <parent link="base_link"/>
+    <child link="laser_frame"/>
+    <origin xyz="0.1 0 0.175" rpy="0 0 0"/>
+  </joint>
+  <xacro:if value="${'$(arg gazebo)' == 'ignition'}">
+    <gazebo reference="laser_frame">
+        <material>Gazebo/Red</material>
+        <sensor name="laser" type="ray">
+            <pose> 0 0 0 0 0 0 </pose>
+            <visualize>true</visualize>
+            <update_rate>10</update_rate>
+            <ray>
+                <scan>
+                    <horizontal>
+                        <samples>360</samples>
+                        <min_angle>-3.14</min_angle>
+                        <max_angle>3.14</max_angle>
+                    </horizontal>
+                </scan>
+                <range>
+                    <min>0.3</min>
+                    <max>12</max>
+                </range>
+            </ray>
+            <plugin name="laser_controller" filename="libgazebo_ros_ray_sensor.so">
+                <ros>
+                    <argument>~/out:=scan</argument>
+                </ros>
+                <output_type>sensor_msgs/LaserScan</output_type>
+                <frame_name>laser_frame</frame_name>
+            </plugin>
+        </sensor>
+    </gazebo>
+  </xacro:if> -->
 </robot>

Commit message: Añadido lidar(con errores) + bridge + renombrar el mundo

File: create3_sim/irobot_create_common/irobot_create_description/urdf/create3.urdf.xacro (robot description, xacro)
@@ -11,4 +11,5 @@
   <xacro:include filename="$(find irobot_create_description)/urdf/sensors/optical_mouse.urdf.xacro"/>
   <xacro:include filename="$(find irobot_create_description)/urdf/wheel_with_wheeldrop.urdf.xacro" />
+  <xacro:include filename="$(find irobot_create_description)/urdf/sensors/lidar_sensor.urdf.xacro" />
   <!-- Gazebo version -->
   <xacro:arg name="gazebo"                       default="classic" />
@@ -268,55 +269,6 @@
   </xacro:if>
   <!-- LIDAR -->
-  <!-- NO FUNCIONA
-  <link name="laser_frame">
-      <visual>
-          <geometry>
-              <cylinder radius="0.05" length="0.04"/>
-          </geometry>
-          <material name="red"/>
-      </visual>
-      <collision>
-          <geometry>
-              <cylinder radius="0.05" length="0.04"/>
-          </geometry>
-      </collision>
-      <xacro:inertial_cylinder mass="0.1" length="0.04" radius="0.05">
-          <origin xyz="0 0 0" rpy="0 0 0"/>
-      </xacro:inertial_cylinder>
-  </link>
-  <joint name="laser_joint" type="fixed">
-    <parent link="base_link"/>
-    <child link="laser_frame"/>
-    <origin xyz="0.1 0 0.175" rpy="0 0 0"/>
-  </joint>
-  <xacro:if value="${'$(arg gazebo)' == 'ignition'}">
-    <gazebo reference="laser_frame">
-        <material>Gazebo/Red</material>
-        <sensor name="laser" type="ray">
-            <pose> 0 0 0 0 0 0 </pose>
-            <visualize>true</visualize>
-            <update_rate>10</update_rate>
-            <ray>
-                <scan>
-                    <horizontal>
-                        <samples>360</samples>
-                        <min_angle>-3.14</min_angle>
-                        <max_angle>3.14</max_angle>
-                    </horizontal>
-                </scan>
-                <range>
-                    <min>0.3</min>
-                    <max>12</max>
-                </range>
-            </ray>
-            <plugin name="laser_controller" filename="libgazebo_ros_ray_sensor.so">
-                <ros>
-                    <argument>~/out:=scan</argument>
-                </ros>
-                <output_type>sensor_msgs/LaserScan</output_type>
-                <frame_name>laser_frame</frame_name>
-            </plugin>
-        </sensor>
-    </gazebo>
-  </xacro:if> -->
+  <xacro:rplidar name="lidar" gazebo="$(arg gazebo)" namespace="$(arg namespace)">
+    <origin xyz="0 0 0.15"  rpy="0 0 0"/>
+  </xacro:rplidar>
 </robot>

Commit message: Lidar funcional +cambio de nombre del mundo a minusculas

File: create3_sim/irobot_create_common/irobot_create_description/urdf/create3.urdf.xacro (robot description, xacro)
@@ -264,5 +264,5 @@
     <gazebo>
       <plugin filename="libgz-sim-sensors-system.so" name="gz::sim::systems::Sensors">
-        <render_engine>ogre</render_engine>
+        <render_engine>ogre2</render_engine>
       </plugin>
     </gazebo>
@@ -270,5 +270,5 @@
   <!-- LIDAR -->
   <xacro:rplidar name="lidar" gazebo="$(arg gazebo)" namespace="$(arg namespace)">
-    <origin xyz="0 0 0.15"  rpy="0 0 0"/>
+    <origin xyz="0 0 0.135"  rpy="0 0 0"/>
   </xacro:rplidar>
 </robot>

File: create3_sim/irobot_create_common/irobot_create_description/urdf/sensors/lidar_sensor.urdf.xacro (robot description, xacro)
@@ -33,4 +33,5 @@
         <pose>0 0 0 0 0 0</pose>
         <update_rate>10.0</update_rate>
+        <gz_frame_id>${name}_link</gz_frame_id>
         <ray>
           <scan>
@@ -48,5 +49,5 @@
           </range>
         </ray>
-        <plugin name="${name}_plugin" filename="gpu_lidar"/>
+        <!-- <plugin name="${name}_plugin" filename="gpu_lidar"/> -->
       </sensor>
       <xacro:material_darkgray/>
